Commit message: Gazebo launch with xacro robot, diff-drive control and ultrasonic sensors

File: xacro/mini_pi.xacro (robot description, xacro)
@@ -2,13 +2,13 @@
 <robot xmlns:xacro="http://www.ros.org/wiki/xacro" name="mini_pi">
   <!-- Colors -->
-  <xacro:include filename="$(find mini_pi_robot_description)/xacro/materials/materials.xacro"/>
+  <xacro:include filename="$(find mini_pi_description)/xacro/materials/materials.xacro"/>
   <!-- Shapes & Caster -->
-  <xacro:include filename="$(find mini_pi_robot_description)/xacro/macros/shapes.xacro"/>
-  <xacro:include filename="$(find mini_pi_robot_description)/xacro/macros/caster.xacro"/>
+  <xacro:include filename="$(find mini_pi_description)/xacro/macros/shapes.xacro"/>
+  <xacro:include filename="$(find mini_pi_description)/xacro/macros/caster.xacro"/>
   <!-- Robot Parts -->
-  <xacro:include filename="$(find mini_pi_robot_description)/xacro/parts/params.xacro"/>
-  <xacro:include filename="$(find mini_pi_robot_description)/xacro/parts/chassis.xacro"/>
-  <xacro:include filename="$(find mini_pi_robot_description)/xacro/parts/wheels.xacro"/>
-  <xacro:include filename="$(find mini_pi_robot_description)/xacro/parts/sensors_ultrasonic.xacro"/>
+  <xacro:include filename="$(find mini_pi_description)/xacro/parts/params.xacro"/>
+  <xacro:include filename="$(find mini_pi_description)/xacro/parts/chassis.xacro"/>
+  <xacro:include filename="$(find mini_pi_description)/xacro/parts/wheels.xacro"/>
+  <xacro:include filename="$(find mini_pi_description)/xacro/parts/sensors_ultrasonic.xacro"/>
   <!-- ============================ -->
   <!-- =   Robot Model Assembly   = -->
@@ -19,5 +19,5 @@
     <parent link="base_footprint"/>
     <child  link="base_link"/>
-    <origin xyz="0 0 0.0585" rpy="0 0 0"/>
+    <origin xyz="0 0 0.0575" rpy="0 0 0"/>
   </joint>
   <!-- Define the base link-->
@@ -35,5 +35,5 @@
     name="front_caster"
     parent_link="base_link"
-    pos_x="0.0400" pos_y="0" pos_z="-0.0495"
+    pos_x="0.0400" pos_y="0" pos_z="-0.0500"
     color_roll="Yellow"
     color_pitch="Pink"
@@ -45,5 +45,5 @@
     name="back_caster"
     parent_link="base_link"
-    pos_x="-0.0400" pos_y="0" pos_z="-0.0495"
+    pos_x="-0.0400" pos_y="0" pos_z="-0.0500"
     color_roll="Yellow"
     color_pitch="Pink"
@@ -52,3 +52,28 @@
     radius="0.0075"
     mass="0.0002"/>
+  <!-- ==== Ros2 Controller ==== -->
+  <ros2_control name="MiniPiSystem" type="system">
+    <hardware>
+      <plugin>gz_ros2_control/GazeboSimSystem</plugin>
+    </hardware>
+    <joint name="wheel_right_joint">
+      <command_interface name="velocity"/>
+      <state_interface name="position"/>
+      <state_interface name="velocity"/>
+    </joint>
+    <joint name="wheel_left_joint">
+      <command_interface name="velocity"/>
+      <state_interface name="position"/>
+      <state_interface name="velocity"/>
+    </joint>
+  </ros2_control>
+  <!-- ==== Gazebo plugin ==== -->
+  <gazebo>
+    <plugin filename="libgz_ros2_control-system.so" name="gz_ros2_control::GazeboSimROS2ControlPlugin">
+      <parameters>$(find mini_pi_description)/config/controller.yaml</parameters>
+    </plugin>
+    <plugin filename="gz-sim-sensors-system" name="gz::sim::systems::Sensors">
+      <render_engine>ogre2</render_engine>
+    </plugin>
+  </gazebo>
 </robot>

File: xacro/parts/sensors_ultrasonic.xacro (robot description, xacro)
@@ -1,4 +1,8 @@
-<?xml version="1.0"?>
 <robot xmlns:xacro="http://www.ros.org/wiki/xacro" name="mini_pi">
+  <!-- Sensor pose: rendering gazebo -->
+  <xacro:property name="ULTRA_FRONT" value="0.0485  0       0.0300  0  0  0" />
+  <xacro:property name="ULTRA_RIGHT" value="0      -0.0485  0.0300  0  0  4.7123" />
+  <xacro:property name="ULTRA_BACK"  value="-0.0485 0       0.0300  0  0  3.14159" />
+  <xacro:property name="ULTRA_LEFT"  value="0       0.0485  0.0300  0  0  1.5708" />
   <xacro:macro name="mini_pi_ultrasonic" params="parent">
     <xacro:square_link
@@ -46,4 +50,145 @@
     rpy="0 0 1.5708"
     joint_type="fixed"/>
+    <!-- Lidar attached directly to base_link (parent) -->
+    <gazebo reference="${parent}">
+      <sensor name="ultra_front" type="gpu_lidar">
+        <pose>${ULTRA_FRONT}</pose>
+        <topic>/ultra_front/scan</topic>
+        <always_on>true</always_on>
+        <visualize>true</visualize>
+        <update_rate>10</update_rate>
+        <ray>
+          <scan>
+            <horizontal>
+              <samples>5</samples>
+              <resolution>1</resolution>
+              <min_angle>-0.12</min_angle>
+              <max_angle>0.12</max_angle>
+            </horizontal>
+            <vertical>
+              <samples>1</samples>
+              <resolution>1</resolution>
+              <min_angle>0.0</min_angle>
+              <max_angle>0.0</max_angle>
+            </vertical>
+          </scan>
+          <range>
+            <min>0.02</min>
+            <max>4.0</max>
+            <resolution>0.01</resolution>
+          </range>
+          <noise>
+            <type>gaussian</type>
+            <mean>0.0</mean>
+            <stddev>0.01</stddev>
+          </noise>
+        </ray>
+      </sensor>
+    </gazebo>
+    <gazebo reference="${parent}">
+      <sensor name="ultra_right" type="gpu_lidar">
+        <pose>${ULTRA_RIGHT}</pose>
+        <topic>/ultra_right/scan</topic>
+        <always_on>true</always_on>
+        <visualize>true</visualize>
+        <update_rate>10</update_rate>
+        <ray>
+          <scan>
+            <horizontal>
+              <samples>5</samples>
+              <resolution>1</resolution>
+              <min_angle>-0.12</min_angle>
+              <max_angle>0.12</max_angle>
+            </horizontal>
+            <vertical>
+              <samples>1</samples>
+              <resolution>1</resolution>
+              <min_angle>0.0</min_angle>
+              <max_angle>0.0</max_angle>
+            </vertical>
+          </scan>
+          <range>
+            <min>0.02</min>
+            <max>4.0</max>
+            <resolution>0.01</resolution>
+          </range>
+          <noise>
+            <type>gaussian</type>
+            <mean>0.0</mean>
+            <stddev>0.01</stddev>
+          </noise>
+        </ray>
+      </sensor>
+    </gazebo>
+    <gazebo reference="${parent}">
+      <sensor name="ultra_back" type="gpu_lidar">
+        <pose>${ULTRA_BACK}</pose>
+        <topic>/ultra_back/scan</topic>
+        <always_on>true</always_on>
+        <visualize>true</visualize>
+        <update_rate>10</update_rate>
+        <ray>
+          <scan>
+            <horizontal>
+              <samples>5</samples>
+              <resolution>1</resolution>
+              <min_angle>-0.12</min_angle>
+              <max_angle>0.12</max_angle>
+            </horizontal>
+            <vertical>
+              <samples>1</samples>
+              <resolution>1</resolution>
+              <min_angle>0.0</min_angle>
+              <max_angle>0.0</max_angle>
+            </vertical>
+          </scan>
+          <range>
+            <min>0.02</min>
+            <max>4.0</max>
+            <resolution>0.01</resolution>
+          </range>
+          <noise>
+            <type>gaussian</type>
+            <mean>0.0</mean>
+            <stddev>0.01</stddev>
+          </noise>
+        </ray>
+      </sensor>
+    </gazebo>
+    <gazebo reference="${parent}">
+      <sensor name="ultra_left" type="gpu_lidar">
+        <pose>${ULTRA_LEFT}</pose>
+        <topic>/ultra_left/scan</topic>
+        <always_on>true</always_on>
+        <visualize>true</visualize>
+        <update_rate>10</update_rate>
+        <ray>
+          <scan>
+            <horizontal>
+              <samples>5</samples>
+              <resolution>1</resolution>
+              <min_angle>-0.12</min_angle>
+              <max_angle>0.12</max_angle>
+            </horizontal>
+            <vertical>
+              <samples>1</samples>
+              <resolution>1</resolution>
+              <min_angle>0.0</min_angle>
+              <max_angle>0.0</max_angle>
+            </vertical>
+          </scan>
+          <range>
+            <min>0.02</min>
+            <max>4.0</max>
+            <resolution>0.01</resolution>
+          </range>
+          <noise>
+            <type>gaussian</type>
+            <mean>0.0</mean>
+            <stddev>0.01</stddev>
+          </noise>
+        </ray>
+      </sensor>
+    </gazebo>
   </xacro:macro>
 </robot>

File: xacro/parts/wheels.xacro (robot description, xacro)
@@ -9,5 +9,5 @@
       mass="${wheel_mass}"
       parent_link="${parent}"
-      xyz="0 -0.0385 -0.0275"
+      xyz="0 -0.0380 -0.0275"
       rpy="0 0 0"
       joint_type="continuous"
@@ -20,5 +20,5 @@
       mass="${wheel_mass}"
       parent_link="${parent}"
-      xyz="0 0.0385 -0.0275"
+      xyz="0 0.0380 -0.0275"
       rpy="0 0 0"
       joint_type="continuous"
